Commit message: aruco lab

File: src/ur3e_hande/ur3e_hande_description/urdf/sensors/camera.urdf.xacro (robot description, xacro)
@@ -21,8 +21,8 @@
     </link>
   <!-- Dummy camera link to reorient sensor frames correctly -->
-  <link name="dummy_camera_link"/>
+  <link name="camera_optical_link"/>
   <joint name="dummy_camera_joint" type="fixed">
     <parent link="camera_link"/>
-    <child link="dummy_camera_link"/>
+    <child link="camera_optical_link"/>
     <origin xyz="0 0 0" rpy="-3.14 -1.57 1.57"/> <!-- only cloud is off; previously: ${-pi/2} 0 ${-pi/2}-->
   </joint>

File: src/ur3e_hande/ur3e_hande_description/urdf/ur3e_hande.urdf.xacro (robot description, xacro)
@@ -54,9 +54,9 @@
       </plugin>
   </gazebo>
-  <gazebo reference="dummy_camera_link">
+  <gazebo reference="camera_optical_link">
       <sensor name="camera" type="rgbd_camera">
         <frame_id>camera_depth_optical_frame</frame_id>
         <camera>
-         <optical_frame_id>dummy_camera_link</optical_frame_id> <!-- Previously: camera_color_optical_frame -->
+         <optical_frame_id>camera_optical_link</optical_frame_id> <!-- Previously: camera_color_optical_frame -->
           <horizontal_fov>1.5707963267948966</horizontal_fov>
           <image>
